File: Electrical/BACKPLANE/12_BCKPLN_FPGA_J008340C.brd (EAGLE design)
At the start: 297 x 52.3 mm, 83 parts, among them J100 BNCBNC-4PIN, J101 BNC, J102 BNCBNC-4PIN, J103 BNC, J104 Battery Jack, M1 XEM7001-OUTLINE, M1A XEM7001-P1, M1B XEM7001-P2, M1C XEM7001-P3, P1 CON14ST2X7_PLUG, P10 CON14ST2X7_PLUG, P11 CON14ST2X7_PLUG, P12 CON14ST2X7_PLUG, P2 CON14ST2X7_PLUG, P3 CON14ST2X7_PLUG, P4 CON14ST2X7_PLUG, P5 CON14ST2X7_PLUG, P6 CON14ST2X7_PLUG, P7 CON14ST2X7_PLUG, P8 CON14ST2X7_PLUG, P9 CON14ST2X7_PLUG, U100 2G17, U101 2G17, U102 AS6C3216A, U103 TPS77033, U104 MAX931, U105 TLP241A(TP1,F, U106 2G17, U107 LP2950CDT-5.0, U108 TLP241A(TP1,F, U109 2G17

Commit message: Update BOMs and boards, add miniFlySong photo
Parts:
- J100, J102: value BNCBNC-4PIN -> BNC-4PIN
- J101, J103: value BNC -> BNC-4PIN
Changed lines of the file:
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@@
 <attribute name="VALUE" x="165.616" y="8.814" size="1.27" layer="28" rot="MR0"/>
 </element>
-<element name="J102" library="STEVES_BU" package="BNC-4PIN" value="BNCBNC-4PIN" x="178.5" y="43.4" smashed="yes" rot="MR90">
+<element name="J102" library="STEVES_BU" package="BNC-4PIN" value="BNC-4PIN" x="178.5" y="43.4" smashed="yes" rot="MR90">
 <attribute name="NAME" x="185.133" y="32.831" size="1.016" layer="26" font="vector" ratio="10" rot="MR0"/>
 <attribute name="VALUE" x="191.817" y="39.713" size="1.27" layer="28" ratio="10" rot="MR90"/>
@@
 <attribute name="VALUE" x="99.416" y="43.914" size="1.27" layer="28" rot="MR0"/>
 </element>
-<element name="J100" library="STEVES_BU" package="BNC-4PIN" value="BNCBNC-4PIN" x="201.8" y="43.35" smashed="yes" rot="MR90">
+<element name="J100" library="STEVES_BU" package="BNC-4PIN" value="BNC-4PIN" x="201.8" y="43.35" smashed="yes" rot="MR90">
 <attribute name="NAME" x="212.831" y="39.917" size="1.016" layer="26" font="vector" ratio="10" rot="MR90"/>
 <attribute name="VALUE" x="215.117" y="39.663" size="1.27" layer="28" ratio="10" rot="MR90"/>
@@
 <attribute name="VALUE" x="97.334" y="43.336" size="1.27" layer="28" rot="MR180"/>
 </element>
-<element name="J103" library="STEVES_BU" package="BNC-4PIN" value="BNC" x="131.75" y="43.45" smashed="yes" rot="MR180">
+<element name="J103" library="STEVES_BU" package="BNC-4PIN" value="BNC-4PIN" x="131.75" y="43.45" smashed="yes" rot="MR180">
 <attribute name="NAME" x="136.567" y="34.219" size="1.016" layer="26" font="vector" ratio="10" rot="MR180"/>
 <attribute name="VALUE" x="128.063" y="30.133" size="1.27" layer="28" ratio="10" rot="MR180"/>
 </element>
-<element name="J101" library="STEVES_BU" package="BNC-4PIN" value="BNC" x="155.25" y="43.35" smashed="yes" rot="MR90">
+<element name="J101" library="STEVES_BU" package="BNC-4PIN" value="BNC-4PIN" x="155.25" y="43.35" smashed="yes" rot="MR90">
 <attribute name="NAME" x="163.783" y="33.081" size="1.016" layer="26" font="vector" ratio="10" rot="MR0"/>
 <attribute name="VALUE" x="168.567" y="39.663" size="1.27" layer="28" ratio="10" rot="MR90"/>
