File: Electrical/BACKPLANE/12_BCKPLN_FPGA_J008340C.sch (EAGLE design)
At the start: 83 parts, among them J100 BNCBNC-4PIN, J101 BNC, J102 BNCBNC-4PIN, J103 BNC, J104 Battery Jack, M1 XEM7001-OUTLINE, M1A XEM7001-P1, M1B XEM7001-P2, M1C XEM7001-P3, P1 CON14ST2X7_PLUG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

Commit message: Update BOMs and boards, add miniFlySong photo
Parts:
- J100, J102: value BNCBNC-4PIN -> BNC-4PIN
- J101, J103: value BNC -> BNC-4PIN
