File: miniFlySong/ECAD/miniFlySong_J010706C.brd (EAGLE design)
At the start: 87 x 38.1 mm, 20 parts, among them J1 BNC, J2 Battery Jack, M1 TEENSY_3.1-3.2_OUTER_ROW, P100 CON14ST2X7_PLUG, T1 PIN2F061.200, T2 PIN2F061.200, U1 MAX931, U2 74AUC1G17DBV, U3 TLP241A(TP1,F, U4 TLP241A(TP1,F

Commit message: Update BOMs and boards, add miniFlySong photo
Parts:
- removed M1: TEENSY_3.1-3.2_OUTER_ROW, Teensy_3_and_LC_Series_Boards_v1.4:TEENSY_3.0-3.2&LC_OUTER_ROW
- added M1-1, M1-2: (no value), SparkFun-Connectors:1X14
Connections:
- removed net AGND: M1.AGND
- removed net VBAT: M1.VBAT
- removed net VIN: M1.VIN
- net 3V3: now also M1-2.3; no longer M1.3.3V, M1.3.3V1
- net BATCNTRL: now also M1-1.2; no longer M1.0
- net CIPO: now also M1-1.14; no longer M1.12
- net COPI: now also M1-1.13; no longer M1.11
- net CS: now also M1-2.13; no longer M1.14/A0
- net GND: now also M1-1.1, M1-2.2; no longer M1.GND, M1.GND1
- net SCLK: now also M1-2.14; no longer M1.13
- net SYNC: now also M1-1.5; no longer M1.3
- net VCHECK: now also M1-1.3; no longer M1.1
Routing:
- net GND: track 6.87 -> 9.34 mm
Changed lines of the file:
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@@
 <setting verticaltext="up"/>
 </settings>
-<grid distance="0.05" unitdist="mm" unit="mm" style="lines" multiple="1" display="yes" altdistance="0.025" altunitdist="inch" altunit="inch"/>
+<grid distance="1" unitdist="mil" unit="mil" style="lines" multiple="1" display="yes" altdistance="0.025" altunitdist="inch" altunit="inch"/>
 <layers>
 <layer number="1" name="Top" color="4" fill="1" visible="yes" active="yes"/>
@@
 </autorouter>
 <elements>
-<element name="M1" library="Teensy_3_and_LC_Series_Boards_v1.4" package="TEENSY_3.0-3.2&amp;LC_OUTER_ROW" value="TEENSY_3.1-3.2_OUTER_ROW" x="41.666" y="26.67" smashed="yes" rot="R90">
-<attribute name="NAME" x="26.426" y="17.272" size="1.016" layer="25" font="vector" rot="R180"/>
-<attribute name="VALUE" x="55.636" y="22.86" size="1.016" layer="27" font="vector" rot="R90"/>
-</element>
 <element name="C2" library="STEVES_BU" package="0603S" value="0.1" x="37.094" y="13.208" smashed="yes" rot="R180">
 <attribute name="NAME" x="38.11" y="14.986" size="1.016" layer="25" font="vector" rot="R180"/>
@@
 <attribute name="VALUE" x="3.07" y="37.58" size="1.778" layer="28" rot="MR90"/>
 </element>
+<element name="M1-2" library="SparkFun-Connectors" package="1X14" value="" x="25.146" y="34.29"/>
+<element name="M1-1" library="SparkFun-Connectors" package="1X14" value="" x="25.146" y="19.05"/>
 </elements>
 <signals>
 <signal name="CS">
-<contactref element="M1" pad="14/A0"/>
 <contactref element="P100" pad="4"/>
 <wire x1="77.099" y1="10.446" x2="75.416" y2="10.446" width="0.4064" layer="1"/>
@@
 <wire x1="71.384" y1="14.478" x2="71.384" y2="17.526" width="0.4064" layer="1"/>
 <wire x1="56.652" y1="25.4" x2="55.636" y2="26.416" width="0.4064" layer="1"/>
-<wire x1="55.636" y1="26.416" x2="55.636" y2="34.29" width="0.4064" layer="1"/>
 <wire x1="56.652" y1="25.4" x2="59.6" y2="25.4" width="0.4064" layer="1"/>
 <wire x1="59.6" y1="25.4" x2="63.4" y2="21.6" width="0.4064" layer="1"/>
 <wire x1="63.4" y1="21.6" x2="67.31" y2="21.6" width="0.4064" layer="1"/>
 <wire x1="67.31" y1="21.6" x2="71.384" y2="17.526" width="0.4064" layer="1"/>
+<contactref element="M1-2" pad="13"/>
+<wire x1="55.636" y1="26.416" x2="55.6386" y2="26.416" width="0.4064" layer="1"/>
+<wire x1="55.6386" y1="26.416" x2="55.626" y2="34.29" width="0.4064" layer="1"/>
 </signal>
 <signal name="SCLK">
-<contactref element="M1" pad="13"/>
 <contactref element="P100" pad="3"/>
 <wire x1="79.893" y1="10.446" x2="79.866" y2="10.946" width="0.4064" layer="1"/>
@@
 <wire x1="75.67" y1="11.716" x2="72.654" y2="14.732" width="0.4064" layer="1"/>
 <wire x1="72.654" y1="14.732" x2="72.654" y2="17.78" width="0.4064" layer="1"/>
-<wire x1="60.208" y1="32.258" x2="58.176" y2="34.29" width="0.4064" layer="1"/>
-<wire x1="60.208" y1="32.258" x2="60.208" y2="26.042" width="0.4064" layer="1"/>
+<wire x1="60.208" y1="32.2656" x2="60.208" y2="26.042" width="0.4064" layer="1"/>
 <wire x1="60.208" y1="26.042" x2="63.7" y2="22.55" width="0.4064" layer="1"/>
 <wire x1="63.7" y1="22.55" x2="67.884" y2="22.55" width="0.4064" layer="1"/>
 <wire x1="67.884" y1="22.55" x2="72.654" y2="17.78" width="0.4064" layer="1"/>
+<contactref element="M1-2" pad="14"/>
+<wire x1="60.208" y1="32.2656" x2="58.166" y2="34.29" width="0.4064" layer="1"/>
 </signal>
 <signal name="CIPO">
-<contactref element="M1" pad="12"/>
 <contactref element="P100" pad="2"/>
 <wire x1="77.099" y1="7.906" x2="75.67" y2="7.906" width="0.4064" layer="1"/>
@@
 <wire x1="70.114" y1="13.462" x2="70.114" y2="17.272" width="0.4064" layer="1"/>
 <wire x1="70.114" y1="17.272" x2="66.812" y2="20.574" width="0.4064" layer="1"/>
-<wire x1="66.812" y1="20.574" x2="59.7" y2="20.574" width="0.4064" layer="1"/>
-<wire x1="59.7" y1="20.574" x2="58.176" y2="19.05" width="0.4064" layer="1"/>
+<wire x1="66.812" y1="20.574" x2="59.694" y2="20.574" width="0.4064" layer="1"/>
+<contactref element="M1-1" pad="14"/>
+<wire x1="59.694" y1="20.574" x2="58.166" y2="19.05" width="0.4064" layer="1"/>
 </signal>
 <signal name="COPI">
-<contactref element="M1" pad="11"/>
 <contactref element="P100" pad="1"/>
 <wire x1="79.893" y1="7.906" x2="78.893" y2="6.763" width="0.4064" layer="1"/>
@@
 <wire x1="58.938" y1="17.272" x2="56.906" y2="17.272" width="0.4064" layer="1"/>
 <wire x1="56.906" y1="17.272" x2="55.636" y2="18.796" width="0.4064" layer="1"/>
-<wire x1="55.636" y1="18.796" x2="55.636" y2="19.05" width="0.4064" layer="1"/>
+<contactref element="M1-1" pad="13"/>
+<wire x1="55.626" y1="19.05" x2="55.636" y2="18.796" width="0" layer="19" extent="1-1"/>
 </signal>
 <signal name="BAT+">
@@
 </signal>
 <signal name="3V3">
-<contactref element="M1" pad="3.3V1"/>
-<contactref element="M1" pad="3.3V"/>
 <contactref element="C2" pad="1"/>
 <contactref element="U2" pad="5"/>
@@
 <wire x1="37.856" y1="12.7" x2="37.856" y2="11.902" width="0.4064" layer="1"/>
 <wire x1="37.856" y1="11.902" x2="38.648" y2="11.11" width="0.4064" layer="1"/>
-<wire x1="30.236" y1="34.29" x2="30.236" y2="31.496" width="0.4064" layer="1"/>
 <wire x1="30.236" y1="31.496" x2="38.491" y2="23.241" width="0.4064" layer="1"/>
-<wire x1="38.491" y1="23.241" x2="39.126" y2="22.606" width="0.4064" layer="1"/>
-<wire x1="39.126" y1="22.606" x2="39.126" y2="13.97" width="0.4064" layer="1"/>
-<wire x1="39.126" y1="13.97" x2="37.856" y2="12.7" width="0.4064" layer="1"/>
-<wire x1="58.176" y1="24.13" x2="53.858" y2="24.13" width="0.4064" layer="16"/>
+<wire x1="38.491" y1="23.241" x2="39.116" y2="22.606" width="0.4064" layer="1"/>
+<wire x1="39.116" y1="13.97" x2="37.856" y2="12.7" width="0.4064" layer="1"/>
 <via x="53.858" y="24.13" extent="1-16" drill="0.381"/>
 <wire x1="53.858" y1="24.13" x2="39.3" y2="24.13" width="0.4064" layer="1"/>
 <wire x1="39.3" y1="24.13" x2="38.491" y2="23.241" width="0.4064" layer="1"/>
-<wire x1="58.176" y1="24.13" x2="63.93" y2="24.13" width="0.4064" layer="16"/>
-<wire x1="63.93" y1="24.13" x2="63.95" y2="24.15" width="0.4064" layer="16"/>
 <via x="63.95" y="24.15" extent="1-16" drill="0.381"/>
 <wire x1="63.95" y1="24.15" x2="68.6" y2="24.15" width="0.4064" layer="1"/>
@@
 <wire x1="74.65" y1="18.1" x2="77.065" y2="18.1" width="0.4064" layer="1"/>
 <wire x1="77.065" y1="18.1" x2="77.099" y2="18.066" width="0.4064" layer="1"/>
+<contactref element="M1-2" pad="3"/>
+<wire x1="39.116" y1="13.97" x2="39.116" y2="22.606" width="0.254" layer="1"/>
+<wire x1="30.236" y1="31.496" x2="30.236" y2="34.28" width="0.4064" layer="1"/>
+<wire x1="30.236" y1="34.28" x2="30.226" y2="34.29" width="0.4064" layer="1"/>
+<wire x1="53.858" y1="24.13" x2="63.93" y2="24.13" width="0.4064" layer="16"/>
+<wire x1="63.93" y1="24.13" x2="63.95" y2="24.15" width="0.4064" layer="16"/>
 </signal>
 <signal name="GND">
-<contactref element="M1" pad="GND"/>
-<contactref element="M1" pad="GND1"/>
 <contactref element="C2" pad="2"/>
 <contactref element="U2" pad="3"/>
@@
 <via x="35.316" y="12.954" extent="1-16" drill="0.381"/>
 <wire x1="35.316" y1="12.954" x2="34.808" y2="12.446" width="0.4064" layer="16"/>
-</signal>
-<signal name="AGND">
-<contactref element="M1" pad="AGND"/>
-</signal>
-<signal name="VBAT">
-<contactref element="M1" pad="VBAT"/>
-</signal>
-<signal name="VIN">
-<contactref element="M1" pad="VIN"/>
+<contactref element="M1-1" pad="1"/>
+<contactref element="M1-2" pad="2"/>
+<wire x1="27.686" y1="34.29" x2="27.7114" y2="34.295" width="0.4064" layer="16"/>
+<wire x1="27.7114" y1="34.295" x2="27.7114" y2="32.9438" width="0.4064" layer="16"/>
+<wire x1="27.686" y1="34.29" x2="27.686" y2="35.3822" width="0.4064" layer="16"/>
 </signal>
 <signal name="SYNC">
-<contactref element="M1" pad="3"/>
 <contactref element="U2" pad="2"/>
 <wire x1="36.058" y1="10.16" x2="34.808" y2="10.16" width="0.4064" layer="1"/>
 <wire x1="34.808" y1="10.16" x2="34.3" y2="10.668" width="0.4064" layer="1"/>
-<wire x1="34.3" y1="10.668" x2="34.3" y2="18.034" width="0.4064" layer="1"/>
-<wire x1="34.3" y1="18.034" x2="35.316" y2="19.05" width="0.4064" layer="1"/>
+<wire x1="34.3" y1="10.668" x2="34.3" y2="18.04" width="0.4064" layer="1"/>
+<contactref element="M1-1" pad="5"/>
+<wire x1="34.3" y1="18.04" x2="35.306" y2="19.05" width="0.4064" layer="1"/>
 </signal>
 <signal name="N$2">
@@
 </signal>
 <signal name="VCHECK">
-<contactref element="M1" pad="1"/>
-<wire x1="30.49" y1="18.796" x2="30.236" y2="19.05" width="0.4064" layer="1"/>
+<contactref element="M1-1" pad="3"/>
 </signal>
 <signal name="N$15">
@@
 </signal>
 <signal name="BATCNTRL">
-<contactref element="M1" pad="0"/>
 <wire x1="24.902" y1="2.286" x2="26.426" y2="3.81" width="0.4064" layer="1"/>
 <wire x1="26.426" y1="3.81" x2="26.426" y2="16.002" width="0.4064" layer="1"/>
 <wire x1="26.426" y1="16.002" x2="27.696" y2="17.272" width="0.4064" layer="1"/>
-<wire x1="27.696" y1="17.272" x2="27.696" y2="19.05" width="0.4064" layer="1"/>
 <contactref element="R7" pad="1"/>
 <wire x1="16.647" y1="2.286" x2="24.902" y2="2.286" width="0.4064" layer="1"/>
+<contactref element="M1-1" pad="2"/>
+<wire x1="27.696" y1="17.272" x2="27.696" y2="19.044" width="0.4064" layer="1"/>
+<wire x1="27.696" y1="19.044" x2="27.686" y2="19.05" width="0.4064" layer="1"/>
 </signal>
 <signal name="N$7">
